Commit message: Update stella.xacro

File: stella_description/urdf/stella.xacro (robot description, xacro)
@@ -17,5 +17,5 @@
       <origin xyz="0 0 ${bodyHeight/2}" rpy="0 0 0"/>
       <geometry>
-        <mesh filename="package://stella_description/meshes/bases/STELLA-N1.stl" scale="0.001 0.001 0.001"/>
+        <mesh filename="package://stella_description/meshes/bases/STELLA-N2.stl" scale="0.001 0.001 0.001"/>
       </geometry>
       <material name="grey"/>

Commit message: Update stella.xacro

File: stella_description/urdf/stella.xacro (robot description, xacro)
@@ -44,5 +44,5 @@
     <parent link="base_link"/>
     <child link="base_scan"/>
-    <origin xyz="${bodyLength/2 - 0.025} 0 ${bodyHeight - 0.024}" rpy="0 0 ${PI}"/>
+    <origin xyz="${bodyLength/2 - 0.025} 0 ${bodyHeight - 0.005}" rpy="0 0 ${PI}"/>
   </joint>
   <link name="base_scan" />
